Commit message: 修复URDF网格路径为ROS2标准格式
- 将左手URDF中的52处相对路径改为package://格式
- 从 filename=palm_mask.STL 改为 filename=package://wujihand-urdf/meshes/left/palm_mask.STL
- 确保RViz/Gazebo能正确加载所有网格模型
- 右手URDF路径已是正确格式，无需修改

File: Description/urdf/left.urdf (robot description, URDF)
Before this commit: robot wujihand-left-v1.0.0, 26 links, 25 joints
Links:
- link finger1_link1: geometry collision mesh filename=package://wujihand-urdf/meshes/left/finger1_link1.STL; visual mesh filename=package://wujihand-urdf/meshes/left/finger1_link1.STL
- link finger1_link2: geometry collision mesh filename=package://wujihand-urdf/meshes/left/finger1_link2.STL; visual mesh filename=package://wujihand-urdf/meshes/left/finger1_link2.STL
- link finger1_link3: geometry collision mesh filename=package://wujihand-urdf/meshes/left/finger1_link3.STL; visual mesh filename=package://wujihand-urdf/meshes/left/finger1_link3.STL
- link finger1_link4: geometry collision mesh filename=package://wujihand-urdf/meshes/left/finger1_link4.STL; visual mesh filename=package://wujihand-urdf/meshes/left/finger1_link4.STL
- link finger1_tip_link: geometry collision mesh filename=package://wujihand-urdf/meshes/left/finger1_tip_link.STL; visual mesh filename=package://wujihand-urdf/meshes/left/finger1_tip_link.STL
- link finger2_link1: geometry collision mesh filename=package://wujihand-urdf/meshes/left/finger2_link1.STL; visual mesh filename=package://wujihand-urdf/meshes/left/finger2_link1.STL
- link finger2_link2: geometry collision mesh filename=package://wujihand-urdf/meshes/left/finger2_link2.STL; visual mesh filename=package://wujihand-urdf/meshes/left/finger2_link2.STL
- link finger2_link3: geometry collision mesh filename=package://wujihand-urdf/meshes/left/finger2_link3.STL; visual mesh filename=package://wujihand-urdf/meshes/left/finger2_link3.STL
- link finger2_link4: geometry collision mesh filename=package://wujihand-urdf/meshes/left/finger2_link4.STL; visual mesh filename=package://wujihand-urdf/meshes/left/finger2_link4.STL
- link finger2_tip_link: geometry collision mesh filename=package://wujihand-urdf/meshes/left/finger2_tip_link.STL; visual mesh filename=package://wujihand-urdf/meshes/left/finger2_tip_link.STL
- link finger3_link1: geometry collision mesh filename=package://wujihand-urdf/meshes/left/finger3_link1.STL; visual mesh filename=package://wujihand-urdf/meshes/left/finger3_link1.STL
- link finger3_link2: geometry collision mesh filename=package://wujihand-urdf/meshes/left/finger3_link2.STL; visual mesh filename=package://wujihand-urdf/meshes/left/finger3_link2.STL
- link finger3_link3: geometry collision mesh filename=package://wujihand-urdf/meshes/left/finger3_link3.STL; visual mesh filename=package://wujihand-urdf/meshes/left/finger3_link3.STL
- link finger3_link4: geometry collision mesh filename=package://wujihand-urdf/meshes/left/finger3_link4.STL; visual mesh filename=package://wujihand-urdf/meshes/left/finger3_link4.STL
- link finger3_tip_link: geometry collision mesh filename=package://wujihand-urdf/meshes/left/finger3_tip_link.STL; visual mesh filename=package://wujihand-urdf/meshes/left/finger3_tip_link.STL
- link finger4_link1: geometry collision mesh filename=package://wujihand-urdf/meshes/left/finger4_link1.STL; visual mesh filename=package://wujihand-urdf/meshes/left/finger4_link1.STL
- link finger4_link2: geometry collision mesh filename=package://wujihand-urdf/meshes/left/finger4_link2.STL; visual mesh filename=package://wujihand-urdf/meshes/left/finger4_link2.STL
- link finger4_link3: geometry collision mesh filename=package://wujihand-urdf/meshes/left/finger4_link3.STL; visual mesh filename=package://wujihand-urdf/meshes/left/finger4_link3.STL
- link finger4_link4: geometry collision mesh filename=package://wujihand-urdf/meshes/left/finger4_link4.STL; visual mesh filename=package://wujihand-urdf/meshes/left/finger4_link4.STL
- link finger4_tip_link: geometry collision mesh filename=package://wujihand-urdf/meshes/left/finger4_tip_link.STL; visual mesh filename=package://wujihand-urdf/meshes/left/finger4_tip_link.STL
- link finger5_link1: geometry collision mesh filename=package://wujihand-urdf/meshes/left/finger5_link1.STL; visual mesh filename=package://wujihand-urdf/meshes/left/finger5_link1.STL
- link finger5_link2: geometry collision mesh filename=package://wujihand-urdf/meshes/left/finger5_link2.STL; visual mesh filename=package://wujihand-urdf/meshes/left/finger5_link2.STL
- link finger5_link3: geometry collision mesh filename=package://wujihand-urdf/meshes/left/finger5_link3.STL; visual mesh filename=package://wujihand-urdf/meshes/left/finger5_link3.STL
- link finger5_link4: geometry collision mesh filename=package://wujihand-urdf/meshes/left/finger5_link4.STL; visual mesh filename=package://wujihand-urdf/meshes/left/finger5_link4.STL
- link finger5_tip_link: geometry collision mesh filename=package://wujihand-urdf/meshes/left/finger5_tip_link.STL; visual mesh filename=package://wujihand-urdf/meshes/left/finger5_tip_link.STL
- link palm_link: geometry collision mesh filename=package://wujihand-urdf/meshes/left/palm_link.STL; visual mesh filename=package://wujihand-urdf/meshes/left/palm_mask.STL

Commit message: 🔧 修复URDF网格路径：添加Description/前缀
问题：URDF路径缺失Description/目录，导致路径不匹配
- 左手URDF：52处路径修复
- 右手URDF：52处路径修复
- 从: package://wujihand-urdf/meshes/left/
- 到: package://wujihand-urdf/Description/meshes/left/

现在所有路径完全匹配实际文件位置 ✓

File: Description/urdf/left.urdf (robot description, URDF)
Before this commit: robot wujihand-left-v1.0.0, 26 links, 25 joints
Links:
- link finger1_link1: geometry collision mesh filename=package://wujihand-urdf/Description/meshes/left/finger1_lin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; visual mesh filename=package://wujihand-urdf/Description/meshes/left/finger1_lin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
- link finger1_link2: geometry collision mesh filename=package://wujihand-urdf/Description/meshes/left/finger1_lin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; visual mesh filename=package://wujihand-urdf/Description/meshes/left/finger1_lin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
- link finger1_link3: geometry collision mesh filename=package://wujihand-urdf/Description/meshes/left/finger1_lin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; visual mesh filename=package://wujihand-urdf/Description/meshes/left/finger1_lin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
- link finger1_link4: geometry collision mesh filename=package://wujihand-urdf/Description/meshes/left/finger1_lin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; visual mesh filename=package://wujihand-urdf/Description/meshes/left/finger1_lin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
- link finger1_tip_link: geometry collision mesh filename=package://wujihand-urdf/Description/meshes/left/finger1_tip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; visual mesh filename=package://wujihand-urdf/Description/meshes/left/finger1_tip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
- link finger2_link1: geometry collision mesh filename=package://wujihand-urdf/Description/meshes/left/finger2_lin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; visual mesh filename=package://wujihand-urdf/Description/meshes/left/finger2_lin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
- link finger2_link2: geometry collision mesh filename=package://wujihand-urdf/Description/meshes/left/finger2_lin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; visual mesh filename=package://wujihand-urdf/Description/meshes/left/finger2_lin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
- link finger2_link3: geometry collision mesh filename=package://wujihand-urdf/Description/meshes/left/finger2_lin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; visual mesh filename=package://wujihand-urdf/Description/meshes/left/finger2_lin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
- link finger2_link4: geometry collision mesh filename=package://wujihand-urdf/Description/meshes/left/finger2_lin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; visual mesh filename=package://wujihand-urdf/Description/meshes/left/finger2_lin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
- link finger2_tip_link: geometry collision mesh filename=package://wujihand-urdf/Description/meshes/left/finger2_tip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; visual mesh filename=package://wujihand-urdf/Description/meshes/left/finger2_tip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
- link finger3_link1: geometry collision mesh filename=package://wujihand-urdf/Description/meshes/left/finger3_lin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; visual mesh filename=package://wujihand-urdf/Description/meshes/left/finger3_lin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
- link finger3_link2: geometry collision mesh filename=package://wujihand-urdf/Description/meshes/left/finger3_lin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; visual mesh filename=package://wujihand-urdf/Description/meshes/left/finger3_lin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
- link finger3_link3: geometry collision mesh filename=package://wujihand-urdf/Description/meshes/left/finger3_lin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; visual mesh filename=package://wujihand-urdf/Description/meshes/left/finger3_lin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
- link finger3_link4: geometry collision mesh filename=package://wujihand-urdf/Description/meshes/left/finger3_lin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; visual mesh filename=package://wujihand-urdf/Description/meshes/left/finger3_lin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
- link finger3_tip_link: geometry collision mesh filename=package://wujihand-urdf/Description/meshes/left/finger3_tip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; visual mesh filename=package://wujihand-urdf/Description/meshes/left/finger3_tip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
- link finger4_link1: geometry collision mesh filename=package://wujihand-urdf/Description/meshes/left/finger4_lin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; visual mesh filename=package://wujihand-urdf/Description/meshes/left/finger4_lin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
- link finger4_link2: geometry collision mesh filename=package://wujihand-urdf/Description/meshes/left/finger4_lin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; visual mesh filename=package://wujihand-urdf/Description/meshes/left/finger4_lin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
- link finger4_link3: geometry collision mesh filename=package://wujihand-urdf/Description/meshes/left/finger4_lin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; visual mesh filename=package://wujihand-urdf/Description/meshes/left/finger4_lin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
- link finger4_link4: geometry collision mesh filename=package://wujihand-urdf/Description/meshes/left/finger4_lin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; visual mesh filename=package://wujihand-urdf/Description/meshes/left/finger4_lin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
- link finger4_tip_link: geometry collision mesh filename=package://wujihand-urdf/Description/meshes/left/finger4_tip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; visual mesh filename=package://wujihand-urdf/Description/meshes/left/finger4_tip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
- link finger5_link1: geometry collision mesh filename=package://wujihand-urdf/Description/meshes/left/finger5_lin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; visual mesh filename=package://wujihand-urdf/Description/meshes/left/finger5_lin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
- link finger5_link2: geometry collision mesh filename=package://wujihand-urdf/Description/meshes/left/finger5_lin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; visual mesh filename=package://wujihand-urdf/Description/meshes/left/finger5_lin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
- link finger5_link3: geometry collision mesh filename=package://wujihand-urdf/Description/meshes/left/finger5_lin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; visual mesh filename=package://wujihand-urdf/Description/meshes/left/finger5_lin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
- link finger5_link4: geometry collision mesh filename=package://wujihand-urdf/Description/meshes/left/finger5_lin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; visual mesh filename=package://wujihand-urdf/Description/meshes/left/finger5_lin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
- link finger5_tip_link: geometry collision mesh filename=package://wujihand-urdf/Description/meshes/left/finger5_tip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; visual mesh filename=package://wujihand-urdf/Description/meshes/left/finger5_tip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
- link palm_link: geometry collision mesh filename=package://wujihand-urdf/Description/meshes/left/palm_link.S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; visual mesh filename=package://wujihand-urdf/Description/meshes/left/palm_mask.S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

File: Description/urdf/right.urdf (robot description, URDF)
Before this commit: robot wujihand-right-v1.0.0, 26 links, 25 joints
Links:
- link finger1_link1: geometry collision mesh filename=package://wujihand-urdf/Description/meshes/right/finger1_li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; visual mesh filename=package://wujihand-urdf/Description/meshes/right/finger1_li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
- link finger1_link2: geometry collision mesh filename=package://wujihand-urdf/Description/meshes/right/finger1_li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; visual mesh filename=package://wujihand-urdf/Description/meshes/right/finger1_li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
- link finger1_link3: geometry collision mesh filename=package://wujihand-urdf/Description/meshes/right/finger1_li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; visual mesh filename=package://wujihand-urdf/Description/meshes/right/finger1_li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
- link finger1_link4: geometry collision mesh filename=package://wujihand-urdf/Description/meshes/right/finger1_li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; visual mesh filename=package://wujihand-urdf/Description/meshes/right/finger1_li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
- link finger1_tip_link: geometry collision mesh filename=package://wujihand-urdf/Description/meshes/right/finger1_ti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; visual mesh filename=package://wujihand-urdf/Description/meshes/right/finger1_ti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
- link finger2_link1: geometry collision mesh filename=package://wujihand-urdf/Description/meshes/right/finger2_li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; visual mesh filename=package://wujihand-urdf/Description/meshes/right/finger2_li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
- link finger2_link2: geometry collision mesh filename=package://wujihand-urdf/Description/meshes/right/finger2_li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; visual mesh filename=package://wujihand-urdf/Description/meshes/right/finger2_li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
- link finger2_link3: geometry collision mesh filename=package://wujihand-urdf/Description/meshes/right/finger2_li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; visual mesh filename=package://wujihand-urdf/Description/meshes/right/finger2_li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
- link finger2_link4: geometry collision mesh filename=package://wujihand-urdf/Description/meshes/right/finger2_li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; visual mesh filename=package://wujihand-urdf/Description/meshes/right/finger2_li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
- link finger2_tip_link: geometry collision mesh filename=package://wujihand-urdf/Description/meshes/right/finger2_ti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; visual mesh filename=package://wujihand-urdf/Description/meshes/right/finger2_ti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
- link finger3_link1: geometry collision mesh filename=package://wujihand-urdf/Description/meshes/right/finger3_li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; visual mesh filename=package://wujihand-urdf/Description/meshes/right/finger3_li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
- link finger3_link2: geometry collision mesh filename=package://wujihand-urdf/Description/meshes/right/finger3_li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; visual mesh filename=package://wujihand-urdf/Description/meshes/right/finger3_li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
- link finger3_link3: geometry collision mesh filename=package://wujihand-urdf/Description/meshes/right/finger3_li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; visual mesh filename=package://wujihand-urdf/Description/meshes/right/finger3_li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
- link finger3_link4: geometry collision mesh filename=package://wujihand-urdf/Description/meshes/right/finger3_li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; visual mesh filename=package://wujihand-urdf/Description/meshes/right/finger3_li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
- link finger3_tip_link: geometry collision mesh filename=package://wujihand-urdf/Description/meshes/right/finger3_ti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; visual mesh filename=package://wujihand-urdf/Description/meshes/right/finger3_ti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
- link finger4_link1: geometry collision mesh filename=package://wujihand-urdf/Description/meshes/right/finger4_li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; visual mesh filename=package://wujihand-urdf/Description/meshes/right/finger4_li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
- link finger4_link2: geometry collision mesh filename=package://wujihand-urdf/Description/meshes/right/finger4_li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; visual mesh filename=package://wujihand-urdf/Description/meshes/right/finger4_li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
- link finger4_link3: geometry collision mesh filename=package://wujihand-urdf/Description/meshes/right/finger4_li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; visual mesh filename=package://wujihand-urdf/Description/meshes/right/finger4_li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
- link finger4_link4: geometry collision mesh filename=package://wujihand-urdf/Description/meshes/right/finger4_li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; visual mesh filename=package://wujihand-urdf/Description/meshes/right/finger4_li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
- link finger4_tip_link: geometry collision mesh filename=package://wujihand-urdf/Description/meshes/right/finger4_ti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; visual mesh filename=package://wujihand-urdf/Description/meshes/right/finger4_ti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
- link finger5_link1: geometry collision mesh filename=package://wujihand-urdf/Description/meshes/right/finger5_li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; visual mesh filename=package://wujihand-urdf/Description/meshes/right/finger5_li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
- link finger5_link2: geometry collision mesh filename=package://wujihand-urdf/Description/meshes/right/finger5_li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; visual mesh filename=package://wujihand-urdf/Description/meshes/right/finger5_li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
- link finger5_link3: geometry collision mesh filename=package://wujihand-urdf/Description/meshes/right/finger5_li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; visual mesh filename=package://wujihand-urdf/Description/meshes/right/finger5_li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
- link finger5_link4: geometry collision mesh filename=package://wujihand-urdf/Description/meshes/right/finger5_li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; visual mesh filename=package://wujihand-urdf/Description/meshes/right/finger5_li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
- link finger5_tip_link: geometry collision mesh filename=package://wujihand-urdf/Description/meshes/right/finger5_ti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; visual mesh filename=package://wujihand-urdf/Description/meshes/right/finger5_ti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
- link palm_link: geometry collision mesh filename=package://wujihand-urdf/Description/meshes/right/palm_link.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; visual mesh filename=package://wujihand-urdf/Description/meshes/right/palm_link.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
